Commit message: readme updated

File: learm_ros2/urdf/learm-gazebo.urdf (robot description, URDF)
Before this commit: robot LeArm, 12 links, 11 joints
Links:
- link base_link: geometry collision mesh filename=file:///home/fushion/Desktop/learm_ros2/src/learm_ros2_desc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; visual mesh filename=file:///home/fushion/Desktop/learm_ros2/src/learm_ros2_desc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
- link finger_left_link: geometry collision mesh filename=file:///home/fushion/Desktop/learm_ros2/src/learm_ros2_desc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; visual mesh filename=file:///home/fushion/Desktop/learm_ros2/src/learm_ros2_desc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
- link finger_right_link: geometry collision mesh filename=file:///home/fushion/Desktop/learm_ros2/src/learm_ros2_desc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; visual mesh filename=file:///home/fushion/Desktop/learm_ros2/src/learm_ros2_desc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
- link forearm_link: geometry collision mesh filename=file:///home/fushion/Desktop/learm_ros2/src/learm_ros2_desc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; visual mesh filename=file:///home/fushion/Desktop/learm_ros2/src/learm_ros2_desc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
- link grip_left_link: geometry collision mesh filename=file:///home/fushion/Desktop/learm_ros2/src/learm_ros2_desc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; visual mesh filename=file:///home/fushion/Desktop/learm_ros2/src/learm_ros2_desc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
- link grip_right_link: geometry collision mesh filename=file:///home/fushion/Desktop/learm_ros2/src/learm_ros2_desc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; visual mesh filename=file:///home/fushion/Desktop/learm_ros2/src/learm_ros2_desc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
- link hand_link: geometry collision mesh filename=file:///home/fushion/Desktop/learm_ros2/src/learm_ros2_desc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; visual mesh filename=file:///home/fushion/Desktop/learm_ros2/src/learm_ros2_desc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
- link humerus_link: geometry collision mesh filename=file:///home/fushion/Desktop/learm_ros2/src/learm_ros2_desc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; visual mesh filename=file:///home/fushion/Desktop/learm_ros2/src/learm_ros2_desc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
- link shoulder_link: geometry collision mesh filename=file:///home/fushion/Desktop/learm_ros2/src/learm_ros2_desc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; visual mesh filename=file:///home/fushion/Desktop/learm_ros2/src/learm_ros2_desc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
- link tendon_left_link: geometry collision mesh filename=file:///home/fushion/Desktop/learm_ros2/src/learm_ros2_desc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; visual mesh filename=file:///home/fushion/Desktop/learm_ros2/src/learm_ros2_desc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
- link tendon_right_link: geometry collision mesh filename=file:///home/fushion/Desktop/learm_ros2/src/learm_ros2_desc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; visual mesh filename=file:///home/fushion/Desktop/learm_ros2/src/learm_ros2_desc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
- link wrist_link: geometry collision mesh filename=file:///home/fushion/Desktop/learm_ros2/src/learm_ros2_desc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; visual mesh filename=file:///home/fushion/Desktop/learm_ros2/src/learm_ros2_desc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
Joints:
- joint wrist_flex: limit lower=-1.57 upper=1.57 effort=1000 velocity=0.5 -> lower=1.57 upper=-1.57 effort=1000 velocity=0.5

File: learm_ros2/urdf/learm-local.urdf (robot description, URDF)
Before this commit: robot LeArm, 12 links, 11 joints
Joints:
- joint wrist_flex: limit lower=-1.57 upper=1.57 effort=1000 velocity=0.5 -> lower=1.57 upper=-1.57 effort=1000 velocity=0.5

File: learm_ros2_description/urdf/learm.urdf (robot description, URDF)
Before this commit: robot learm, 12 links, 11 joints
Joints:
- joint wrist_flex: axis 0 -1 0 -> 0 1 0; limit lower=-1.57 upper=1.57 effort=1000 velocity=0.5 -> lower=1.57 upper=-1.57 effort=1000 velocity=0.5

File: learm_ros2_description/urdf/learm.urdf.xacro (robot description, xacro)
@@ -116,5 +116,5 @@
     <origin xyz="0 0 0.090"/>
     <axis xyz="0 -1 0"/>
-    <limit effort="1000" lower="-1.57" upper="1.57" velocity="0.5"/>
+    <limit effort="1000" lower="1.57" upper="-1.57" velocity="0.5"/>
   </joint>
   <joint name="wrist_roll" type="revolute">
